File: line_injector.kicad_pcb (KiCad board)
At the start: 2 copper layers, 120 x 100 mm, 21 parts, among them J1 Conn_01x01_Female, J2 Conn_01x01_Female, J3 Conn_01x01_Female, J4 Conn_01x01_Female, J5 Conn_01x01_Female, J6 Conn_01x01_Female, J7 Conn_Coaxial, Q1 AOT2618

Commit message: Udpated license to CERN-OHL-W
Other:
- board text added: "Line injector v1.0.2 Design: Patrick Baus Date: 2024-11 https://github.com/PatrickBaus"
- board text removed: "Line injector v1.0.2 Design: Patrick Baus Date: 2024-11 https://github.com/TU-Darmstadt-APQ"
Changed lines of the file:
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@@
 		(rev "v1.0.2")
 		(comment 1 "Copyright (©) 2024, Patrick Baus <patrick.baus@physik.tu-darmstadt.de>")
-		(comment 2 "Licensed under CERN OHL v.1.2")
+		(comment 2 "Licensed under CERN OHL-W v2.0")
 	)
 	(layers
@@
 		(fp_arc
 			(start -17.691791 -12.749206)
-			(mid -16.926426 -12.74787)
+			(mid -16.926425 -12.74787)
 			(end -16.386175 -12.20573)
 			(stroke
@@
 		(fp_arc
 			(start 19.058317 -9.075185)
-			(mid 19.74445 -9.414242)
+			(mid 19.74446 -9.41424)
 			(end 20.469421 -9.168911)
 			(stroke
@@
 		(fp_arc
 			(start 12.79953 -11.8)
-			(mid 13.004551 -12.294999)
+			(mid 13.004541 -12.294989)
 			(end 13.49953 -12.5)
 			(stroke
@@
 		(fp_arc
 			(start 13.725181 -12.49953)
-			(mid 14.203509 -12.285818)
+			(mid 14.203536 -12.285845)
 			(end 14.39953 -11.8)
 			(stroke
@@
 		(fp_arc
 			(start 14.30047 11.8)
-			(mid 14.095449 12.294999)
+			(mid 14.095459 12.294989)
 			(end 13.60047 12.5)
 			(stroke
@@
 		)
 	)
-	(gr_text "Line injector v1.0.2\nDesign: Patrick Baus\nDate: 2024-11\nhttps://github.com/TU-Darmstadt-APQ"
+	(gr_text "Line injector v1.0.2\nDesign: Patrick Baus\nDate: 2024-11\nhttps://github.com/PatrickBaus"
 		(at 100.06 43.355 0)
 		(layer "F.SilkS")
