File: line_injector.kicad_sch (KiCad schematic)
At the start: 22 parts, among them J1 Conn_01x01_Female, J2 Conn_01x01_Female, J3 Conn_01x01_Female, J4 Conn_01x01_Female, J5 Conn_01x01_Female, J6 Conn_01x01_Female, J7 Conn_Coaxial, Q1 AOT2618

Commit message: Added RoHS info
Added temperature data
Parts:
- C1, C3: RoHS (none) -> Yes; Temperature (none) -> Tstorage = –55 °C to 105 °C
- C2, C4, C6: RoHS (none) -> Yes; Temperature (none) -> Tstorage = –55 °C to 125 °C
- C5: RoHS (none) -> Yes; Temperature (none) -> Tstorage = –40 °C to 125 °C
- HS1, N1: RoHS (none) -> Yes
- J1, J2, J3, J5, J6: RoHS (none) -> Yes; Temperature (none) -> Tstorage = –25 °C to 80 °C, FCR7350X: -40 °C to 80 °C
- J4: RoHS (none) -> Yes; Tempeature (none) -> Tstorage = –25 °C to 80 °C, FCR7350X: -40 °C to 80 °C; Temperature (none) -> Tstorage = –25 °C to 80 °C, FCR7350X: -40 °C to 80 °C
- J7: RoHS (none) -> By excemption; Temperature (none) -> Tstorage = –55 °C to 85 °C
- Q1: RoHS (none) -> Yes; Temperature (none) -> Tstorage = –55 °C to 175 °C
- R1, R2, R3, R4: RoHS (none) -> By excemption; Temperature (none) -> Tstorage = –55 °C to 155 °C
